File: lora-bone.kicad_pcb (KiCad board)
At the start: 2 copper layers, 30 x 98 mm, 30 parts, among them J1 Analog IN, J10 GS2, J11 GS2, J12 GS2, J13 GS2, J14 POWER OUT, J2 POWER, J3 Bluepill left, J4 PWM OUT, J5 SPI OUT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

Commit message: Exported components diagramm as svg
Parts:
- removed the G*** at (46.5, 70.6)
